File: euclid36.kicad_pcb (KiCad board)
At the start: 2 copper layers, 248.2 x 127 mm, 94 parts, among them SW10 SW_PUSH, SW11 SW_PUSH, SW12 SW_PUSH, SW14 SW_PUSH, SW15 SW_PUSH, SW16 SW_PUSH, SW17 SW_PUSH, SW18 SW_PUSH, SW19 SW_PUSH, SW2 SW_PUSH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

Commit message: Added one more hole for another stabilizer in the center
Parts:
- added REF**: M2_Hole_NPTH_Outside, _reviung-kbd:M2_Hole_NPTH_Outside, F.Cu at (153.2, 87.4)
