File: mx-v2/_autosave-euclid36.sch (KiCad schematic (older format))
At the start: 114 parts, among them SW1 RotaryEncoder_Switch, SW10 SW_PUSH, SW11 SW_PUSH, SW12 SW_PUSH, SW14 SW_PUSH, SW15 SW_PUSH, SW16 SW_PUSH, SW17 SW_PUSH, SW18 SW_PUSH, SW19 SW_PUSH, SW2 SW_PUSH, SW20 SW_PUSH, SW21 SW_PUSH, SW22 SW_PUSH, SW23 SW_PUSH, SW25 SW_PUSH, SW26 SW_PUSH, SW27 SW_PUSH, SW28 SW_PUSH, SW29 SW_PUSH, SW3 SW_PUSH, SW31 SW_PUSH, SW32 SW_PUSH, SW33 SW_PUSH, SW34 SW_PUSH, SW35 SW_PUSH, SW37 SW_PUSH, SW38 SW_PUSH, SW39 SW_PUSH, SW4 SW_PUSH, SW40 SW_PUSH, SW41 SW_PUSH, SW42 SW_PUSH, SW5 SW_PUSH, SW6 SW_PUSH, SW7 RotaryEncoder_Switch, SW8 SW_PUSH, SW9 SW_PUSH, U1 USBLC6-2SC6, U2 ATmega32U4-AU, Y1 XTAL

Commit message: Added support for two joysticks, but can't use both at the same time, as they share pins
Connections:
- net GND: now also S1.H3 (H-), S1.V3 (V-); no longer S1.H1 (H+), S1.V1 (V+)
- net VCC: now also S1.H1 (H+), S1.V1 (V+); no longer S1.H3 (H-), S1.V3 (V-)
Changed lines of the file:
@@
 L power:GND #PWR0118
 U 1 1 609CC72A
-P 3150 750
-F 0 "#PWR0118" H 3150 500 50  0001 C CNN
-F 1 "GND" V 3155 622 50  0000 R CNN
-F 2 "" H 3150 750 50  0001 C CNN
-F 3 "" H 3150 750 50  0001 C CNN
-	1    3150 750
+P 3150 950
+F 0 "#PWR0118" H 3150 700 50  0001 C CNN
+F 1 "GND" V 3155 822 50  0000 R CNN
+F 2 "" H 3150 950 50  0001 C CNN
+F 3 "" H 3150 950 50  0001 C CNN
+	1    3150 950
 	0    1    1    0
 $EndComp
@@
 L power:VCC #PWR0119
 U 1 1 609CD529
-P 3150 950
-F 0 "#PWR0119" H 3150 800 50  0001 C CNN
-F 1 "VCC" V 3165 1077 50  0000 L CNN
-F 2 "" H 3150 950 50  0001 C CNN
-F 3 "" H 3150 950 50  0001 C CNN
-	1    3150 950
+P 3150 750
+F 0 "#PWR0119" H 3150 600 50  0001 C CNN
+F 1 "VCC" V 3165 877 50  0000 L CNN
+F 2 "" H 3150 750 50  0001 C CNN
+F 3 "" H 3150 750 50  0001 C CNN
+	1    3150 750
 	0    -1   -1   0
 $EndComp
@@
 L power:VCC #PWR0120
 U 1 1 609CDAB2
-P 3150 1350
-F 0 "#PWR0120" H 3150 1200 50  0001 C CNN
-F 1 "VCC" V 3165 1477 50  0000 L CNN
-F 2 "" H 3150 1350 50  0001 C CNN
-F 3 "" H 3150 1350 50  0001 C CNN
-	1    3150 1350
+P 3150 1150
+F 0 "#PWR0120" H 3150 1000 50  0001 C CNN
+F 1 "VCC" V 3165 1277 50  0000 L CNN
+F 2 "" H 3150 1150 50  0001 C CNN
+F 3 "" H 3150 1150 50  0001 C CNN
+	1    3150 1150
 	0    -1   -1   0
 $EndComp
@@
 L power:GND #PWR0121
 U 1 1 609CDE10
-P 3150 1150
-F 0 "#PWR0121" H 3150 900 50  0001 C CNN
-F 1 "GND" V 3155 1022 50  0000 R CNN
-F 2 "" H 3150 1150 50  0001 C CNN
-F 3 "" H 3150 1150 50  0001 C CNN
-	1    3150 1150
+P 3150 1350
+F 0 "#PWR0121" H 3150 1100 50  0001 C CNN
+F 1 "GND" V 3155 1222 50  0000 R CNN
+F 2 "" H 3150 1350 50  0001 C CNN
+F 3 "" H 3150 1350 50  0001 C CNN
+	1    3150 1350
 	0    1    1    0
 $EndComp
@@
 Connection ~ 2650 2550
 $Comp
-L power:GND #PWR?
+L power:GND #PWR0122
 U 1 1 60BD365C
 P 3150 1650
-F 0 "#PWR?" H 3150 1400 50  0001 C CNN
+F 0 "#PWR0122" H 3150 1400 50  0001 C CNN
 F 1 "GND" V 3155 1522 50  0000 R CNN
 F 2 "" H 3150 1650 50  0001 C CNN
